Commit message: docs: refine ROS2 navigation study notes structure

File: projects/ros2_navigation_lab/src/lee_robot_description/urdf/turtlebot.xacro (robot description, xacro)
@@ -1,4 +1,6 @@
 <?xml version="1.0"?>
 <robot xmlns:xacro="http://www.ros.org/wiki/xacro" name="turtlebot">
+  <xacro:arg name="namespace" default="lee"/>
+  <xacro:arg name="odom_frame" default="odom_lee"/>
   <!-- ========== MATERIALS ========== -->
   <material name="black">

File: projects/ros2_navigation_lab/src/lee_robot_description/urdf/turtlebot_gaze.xacro (robot description, xacro)
@@ -1,4 +1,7 @@
 <?xml version="1.0"?>
 <robot xmlns:xacro="http://www.ros.org/wiki/xacro">
+  <xacro:arg name="namespace" default="lee"/>
+  <xacro:arg name="odom_frame" default="odom_lee"/>
+  <xacro:property name="robot_namespace" value="/$(arg namespace)"/>
   <!-- ========== Physical Properties ========== -->
   <gazebo reference="base_link">
@@ -32,7 +35,7 @@
     <plugin name="diff_drive" filename="libgazebo_ros_diff_drive.so">
       <ros>
-        <namespace>/lee</namespace>
-        <remapping>/tf:=/lee/tf</remapping>
-        <remapping>/tf_static:=/lee/tf_static</remapping>
+        <namespace>${robot_namespace}</namespace>
+        <remapping>/tf:=${robot_namespace}/tf</remapping>
+        <remapping>/tf_static:=${robot_namespace}/tf_static</remapping>
       </ros>
       <update_rate>50.0</update_rate>
@@ -53,5 +56,5 @@
       <publish_wheel_tf>false</publish_wheel_tf>
       <!-- Coordinate Frames -->
-      <odometry_frame>odom_lee</odometry_frame>
+      <odometry_frame>$(arg odom_frame)</odometry_frame>
       <robot_base_frame>base_footprint</robot_base_frame>
     </plugin>
@@ -61,5 +64,5 @@
     <plugin name="gazebo_ros_joint_state_publisher" filename="libgazebo_ros_joint_state_publisher.so">
       <ros>
-        <namespace>/lee</namespace>
+        <namespace>${robot_namespace}</namespace>
       </ros>
       <update_rate>30.0</update_rate>
@@ -91,5 +94,5 @@
       <plugin name="laser_controller" filename="libgazebo_ros_ray_sensor.so">
         <ros>
-          <namespace>/lee</namespace>
+          <namespace>${robot_namespace}</namespace>
           <remapping>~/out:=scan</remapping>
         </ros>
@@ -148,5 +151,5 @@
       <plugin name="imu_plugin" filename="libgazebo_ros_imu_sensor.so">
         <ros>
-          <namespace>/lee</namespace>
+          <namespace>${robot_namespace}</namespace>
           <remapping>~/out:=imu</remapping>
         </ros>
@@ -175,7 +178,7 @@
       <plugin name="camera_controller" filename="libgazebo_ros_camera.so">
         <ros>
-          <namespace>/lee</namespace>
-          <remapping>/lee/camera/image_raw:=/lee/image_raw</remapping>
-          <remapping>/lee/camera/camera_info:=/lee/camera_info</remapping>
+          <namespace>${robot_namespace}</namespace>
+          <remapping>${robot_namespace}/camera/image_raw:=${robot_namespace}/image_raw</remapping>
+          <remapping>${robot_namespace}/camera/camera_info:=${robot_namespace}/camera_info</remapping>
         </ros>
         <camera_name>camera</camera_name>
